File: Esp32.kicad_pcb (KiCad board)
At the start: 4 copper layers, 44 parts, among them J1 Conn_01x02, SW1 TS-1088-AR02016, SW2 TS-1088-AR02016, U1 ESP32-S3, U2 AP2114H-3.3TRG1, U3 TPS2116DRL, U4 TP4056-42-ESOP8, U5 TVS, U6 TVS, U7 TVS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

Commit message: kicad-sync: 2026-06-08T04:30:39Z on gaming
Parts:
- removed J1: Conn_01x02, JST:JST_GH_BM02B-GHS-TBT_1x02-1MP_P1.25mm_Vertical
- added TP1: BAT+, TestPoint:TestPoint_Pad_D1.5mm, F.Cu at (173.0, 96.5)
- added TP2: BAT-, TestPoint:TestPoint_Pad_D1.5mm, F.Cu at (173.0, 99.5)
- C1, C10, C11, C12, C13, C15, C16, C17, C18, C2, C3, C4, C5, C6, C7, C8, C9: footprint Capacitor_SMD:C_0402_1005Metric_Pad0.74x0.62mm_HandSolder -> Capacitor_SMD:C_0402_1005Metric
- C14: value 10uf -> 10u; footprint Capacitor_SMD:C_0402_1005Metric_Pad0.74x0.62mm_HandSolder -> Capacitor_SMD:C_0402_1005Metric
- L1, R1, R10, R11, R12, R2, R3, R4, R5, R6, R7, R8, R9: footprint Resistor_SMD:R_0402_1005Metric_Pad0.72x0.64mm_HandSolder -> Resistor_SMD:R_0402_1005Metric
- moved R7 115.0 mm to (175.8, 90.8), turned to 180 degrees
- moved R8 113.4 mm to (175.8, 89.7), turned to 180 degrees
- moved C5 107.5 mm to (174.2, 93.3), turned to 180 degrees
- moved R6 107.3 mm to (166.7, 88.7), turned to 90 degrees
- moved C4 103.3 mm to (167.7, 93.3), turned to 180 degrees
- moved U4 91.2 mm to (170.9, 90.2)
- moved C2 74.8 mm to (164.5, 85.2), turned to 90 degrees
- moved U3 73.4 mm to (160.1, 91.3), turned to -90 degrees
- moved C1 67.6 mm to (156.8, 85.2), turned to -90 degrees
- moved C3 62.7 mm to (158.1, 93.0), turned to 90 degrees
- moved SW1 62.4 mm to (173.5, 69.0), turned to 180 degrees
- moved U2 61.9 mm to (160.7, 84.4), turned to -90 degrees
- moved R5 61.0 mm to (162.1, 91.8), turned to 90 degrees
- moved USB1 58.9 mm to (164.4, 97.1), turned to 0 degrees
- moved U7 57.9 mm to (170.0, 94.0)
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Connections:
- U1 pad 15: unconnected-(U1-GPIO10-Pad15) -> /SRC_STAT(GPOI)
- U1 pad 21: /CHRD_STAT(GPIO) -> /STDBY_STAT(GPIO)
- U1 pad 22: /STDBY_STAT(GPIO) -> /CHRD_STAT(GPIO)
- U1 pad 27: /SRC_STAT(GPOI) -> unconnected-(U1-GPIO21-Pad27)
Routing:
- net /BAT+: track 0.00 -> 24.2 mm, vias 0 -> 2
- net /Boot: track 0.00 -> 18.2 mm, vias 0 -> 3
- net /STDBY_STAT(GPIO): track 0.00 -> 16.3 mm, vias 0 -> 2
- net /D-: track 3.99 -> 18.0 mm
- net /D+: track 4.84 -> 18.8 mm
- net /SRC_STAT(GPOI): track 0.00 -> 13.1 mm, vias 0 -> 2
- net /VBUS_USB: track 0.00 -> 13.0 mm, vias 0 -> 5
- net GND: track 0.00 -> 12.8 mm, vias 0 -> 38
- net /CHIP_PU: track 0.00 -> 11.4 mm, vias 0 -> 2
- net /CHRD_STAT(GPIO): track 0.00 -> 11.4 mm, vias 0 -> 2
- net /VSYS: track 0.00 -> 9.66 mm
- net /XTAL_N: track 0.00 -> 7.68 mm
- net /XTAL_P: track 0.00 -> 5.71 mm
- net /LNA_IN: track 0.00 -> 4.47 mm
- net Net-(U3-PR1): track 0.00 -> 2.44 mm
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- added copper zone on F.Cu, net /3V3
- added copper zone on In2.Cu, net /3V3
- added copper zone on F.Cu, net /Boot
- added copper zone on F.Cu, net /CHIP_PU
- added copper zone on B.Cu, net /VBUS_USB
- added copper zone on F.Cu, net /VBUS_USB
- added copper zone on B.Cu, net GND
- added copper zone on F.Cu, net GND
- added copper zone on In1.Cu, net GND
Other:
- board outline added: 21 x 35.1 mm
