File: Esp32.kicad_sch (KiCad schematic)
At the start: 0 parts

Commit message: Add USB-C connector with CC pulldowns + datasheet
USB1 (TYPE-C 16PIN 2MD) placed and verified via netlist:
- D+ net: U1.26 (GPIO20) + USB1.A6/B6 (Dp1/Dp2)
- D- net: U1.25 (GPIO19) + USB1.A7/B7 (Dn1/Dn2)
- CC1/CC2 pulled down via R1/R2 (5.1k each) to GND
- GND on shield (13/14), A1B12, B1A12, U1.57 EP

Still open at USB block: VBUS feed to LDO, ESD protection on D+/D-.
Datasheets/ PDF added (was missing from prior commit).
netlist.xml + erc.txt gitignored as regenerated artifacts.
Parts:
- added R1, R2: 5.1k, symbol Device:R
- added U1: ESP32-S3, EasyEDA:QFN-56_L7.0-W7.0-P0.40-TL-EP4.0, symbol EasyEDA:ESP32-S3
- added USB1: TYPE-C 16PIN 2MD, EasyEDA:USB-C-SMD_TYPE-C-16PIN-2MD-073, symbol EasyEDA:TYPE-C16PIN2MD
Connections:
- new net: R2.2, USB1.B5 (CC2)
- new net: R1.2, USB1.A5 (CC1)
- new net D+: U1.26 (GPIO20), USB1.A6 (Dp1), USB1.B6 (Dp2)
- new net D-: U1.25 (GPIO19), USB1.A7 (Dn1), USB1.B7 (Dn2)
- new net GND: R1.1, R2.1, U1.57 (EP), USB1.13 (EH), USB1.14 (EH), USB1.A1B12 (GND), USB1.B1A12 (GND)
- new net VBUS_USB: USB1.A4B9 (VBUS), USB1.B4A9 (VBUS)

Commit message: kicad-sync: 2026-06-04T20:56:02Z on Mac
Parts:
- added C1, C2: 4.7u, Capacitor_SMD:C_0402_1005Metric_Pad0.74x0.62mm_HandSolder, symbol Device:C
- added C10, C11: 1u, Capacitor_SMD:C_0402_1005Metric_Pad0.74x0.62mm_HandSolder, symbol Device:C
- added C12, C13, C6, C7, C8, C9: 0.1u, Capacitor_SMD:C_0402_1005Metric_Pad0.74x0.62mm_HandSolder, symbol Device:C
- added C14: 10uf, Capacitor_SMD:C_0402_1005Metric_Pad0.74x0.62mm_HandSolder, symbol Device:C
- added C15, C16: 12p, Capacitor_SMD:C_0402_1005Metric_Pad0.74x0.62mm_HandSolder, symbol Device:C
- added C17, C18: DNP, Capacitor_SMD:C_0402_1005Metric_Pad0.74x0.62mm_HandSolder, symbol Device:C
- added C3, C4, C5: 10u, Capacitor_SMD:C_0402_1005Metric_Pad0.74x0.62mm_HandSolder, symbol Device:C
- added J1: Conn_01x02, JST:JST_GH_BM02B-GHS-TBT_1x02-1MP_P1.25mm_Vertical, symbol Connector_Generic:Conn_01x02
- added L1: 0Ohm, Resistor_SMD:R_0402_1005Metric_Pad0.72x0.64mm_HandSolder, symbol Device:L
- added R10, R11, R12, R9: 10k, Resistor_SMD:R_0402_1005Metric_Pad0.72x0.64mm_HandSolder, symbol Device:R
- added R3: 300k, Resistor_SMD:R_0402_1005Metric_Pad0.72x0.64mm_HandSolder, symbol Device:R
- added R4, R5, R7, R8: 100k, Resistor_SMD:R_0402_1005Metric_Pad0.72x0.64mm_HandSolder, symbol Device:R
- added R6: 2.4k, Resistor_SMD:R_0402_1005Metric_Pad0.72x0.64mm_HandSolder, symbol Device:R
- added RF1: KH-IPEX-K501-29, EasyEDA:ANT-SMD_KH-IPEX-K501-29, symbol EasyEDA:KH-IPEX-K501-29
- added SW1, SW2: TS-1088-AR02016, EasyEDA:SW-SMD_L3.9-W3.0-P4.45, symbol EasyEDA:TS-1088-AR02016
- added U2: AP2114H-3.3TRG1, EasyEDA:SOT-223_L6.7-W3.5-P2.30-BR, symbol EasyEDA:AP2114H-3.3TRG1
- added U3: TPS2116DRL, Package_TO_SOT_SMD:SOT-583-8, symbol Power_Management:TPS2116DRL
- added U4: TP4056-42-ESOP8, Package_SO:SOIC-8-1EP_3.9x4.9mm_P1.27mm_EP2.41x3.3mm_ThermalVias, symbol Battery_Management:TP4056-42-ESOP8
- added U5, U6, U7: TVS, EasyEDA:D0402-BI, symbol EasyEDA:RCLAMP0521P.TCT_C3029033
- added X1: XTM32040000DT00351001, EasyEDA:CRYSTAL-SMD_4P-L3.2-W2.5-BL-2, symbol EasyEDA:XTM32040000DT00351001
- R1, R2: footprint (none) -> Resistor_SMD:R_0402_1005Metric_Pad0.72x0.64mm_HandSolder
Connections:
- net D+: now also U6.1
- net D-: now also U5.1
- net GND: now also C1.2, C10.1, C11.2, C12.1, C13.2, C14.2, C15.2, C16.1, C17.2, C18.2, C2.2, C3.1, C4.1, C5.2, C6.2, C7.2, C8.1, C9.1, J1.2 (Pin_2), R10.2, R11.1, R4.1, R6.2, RF1.1 (GND), RF1.2 (GND), RF1.3 (GND), SW1.1, SW2.1, U2.1 (GND), U3.1 (GND), U4.1 (TEMP), U4.3 (GND), U4.9 (EPAD), U5.2, U6.2, U7.2, X1.2 (GND), X1.4 (GND)
- net VBUS_USB: now also C3.2, C4.2, R3.1, U3.3 (VIN1), U3.5 (MODE), U4.4 (V_{CC}), U4.8 (CE), U7.1
- net LNA_IN: now reaches U1.1 (LNA_IN)
- net LNA_IN: now also C18.1, L1.1
- net 3V3: now reaches U1.2 (VDD3P3)
- net 3V3: now also U1.20 (VDD3P3_RTC), U1.3 (VDD3P3), U1.46 (VDD3P3_CPU), U1.55 (VDDA), U1.56 (VDDA), C1.1, C12.2, C13.1, C14.1, C6.1, C7.1, C8.2, C9.2, R12.1, R5.2, R7.1, R8.1, R9.1, U2.2 (VOUT), U2.4 (VOUT)
- net CHRD_STAT(GPIO): now reaches U1.21 (XTAL_32K_P)
- net CHRD_STAT(GPIO): now also R8.2, U4.7 (~{CHRG})
- net STDBY_STAT(GPIO): now reaches U1.22 (XTAL_32K_N)
- net STDBY_STAT(GPIO): now also R7.2, U4.6 (~{STDBY})
- net SRC_STAT(GPOI): now reaches U1.27 (GPIO21)
- net SRC_STAT(GPOI): now also R5.1, U3.8 (ST)
- net at U1.29 (VDD_SPI): now also C10.2
- net CHIP_PU: now reaches U1.4 (CHIP_PU)
- net CHIP_PU: now also C11.1, R9.2, SW1.2
- net Boot: now reaches U1.5 (GPIO0)
- net Boot: now also R12.2, SW2.2
- net at U1.51 (GPIO45): now also R10.1
- net XTAL_N: now reaches U1.53 (XTAL_N)
- net XTAL_N: now also C16.2, X1.3
- net XTAL_P: now reaches U1.54 (XTAL_P)
- net XTAL_P: now also C15.1, X1.1
- net at U1.8 (GPIO3): now also R11.2
- new net: R3.2, R4.2, U3.4 (PR1)
- new net: C17.1, L1.2, RF1.4 (SIG)
- new net: R6.1, U4.2 (PROG)
- new net BAT+: C5.1, J1.1 (Pin_1), U3.6 (VIN2), U4.5 (BAT)
- new net VSYS: C2.1, U2.3 (VIN), U3.2 (VOUT), U3.7 (VOUT)
- no-connect marks 0 -> 39
Other:
- moved on the sheet: R1, R2, U1, USB1

Commit message: kicad-sync: 2026-06-08T04:30:39Z on gaming
Parts:
- removed J1: Conn_01x02, JST:JST_GH_BM02B-GHS-TBT_1x02-1MP_P1.25mm_Vertical, symbol Connector_Generic:Conn_01x02
- added TP1: BAT+, TestPoint:TestPoint_Pad_D1.5mm, symbol Connector:TestPoint
- added TP2: BAT-, TestPoint:TestPoint_Pad_D1.5mm, symbol Connector:TestPoint
- C1, C10, C11, C12, C13, C15, C16, C17, C18, C2, C3, C4, C5, C6, C7, C8, C9: footprint Capacitor_SMD:C_0402_1005Metric_Pad0.74x0.62mm_HandSolder -> Capacitor_SMD:C_0402_1005Metric
- C14: value 10uf -> 10u; footprint Capacitor_SMD:C_0402_1005Metric_Pad0.74x0.62mm_HandSolder -> Capacitor_SMD:C_0402_1005Metric
- L1, R1, R10, R11, R12, R2, R3, R4, R5, R6, R7, R8, R9: footprint Resistor_SMD:R_0402_1005Metric_Pad0.72x0.64mm_HandSolder -> Resistor_SMD:R_0402_1005Metric
Connections:
- net BAT+: now also TP1.1
- net CHRD_STAT(GPIO): now also U1.22 (XTAL_32K_N); no longer U1.21 (XTAL_32K_P)
- net GND: now also TP2.1
- net SRC_STAT(GPOI): now also U1.15 (GPIO10); no longer U1.27 (GPIO21)
- net STDBY_STAT(GPIO): now also U1.21 (XTAL_32K_P); no longer U1.22 (XTAL_32K_N)
